Commit message: Feat: update kistar urdf (primitive collision)

File: grasp_generation/kistar/kistar_basic_primitiv.urdf (robot description, URDF)
Before this commit: robot kistar_hand, 33 links, 32 joints
Links:
- removed link index_sensor_0
- removed link index_sensor_1
- removed link index_sensor_2
- removed link middle_sensor_0
- removed link middle_sensor_1
- removed link middle_sensor_2
- removed link ring_sensor_0
- removed link ring_sensor_1
- removed link ring_sensor_2
- removed link thumb_sensor_0
- removed link thumb_sensor_1
- link index_basemotor: geometry visual mesh filename=meshes/kistar/finger_basemotor.STL
- link index_link_0: geometry collision box size=0.026000000536441803 0.026000000536441803 0.028453040402382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; visual mesh filename=meshes/kistar/finger_link_0.STL
- link index_link_1: geometry collision box size=0.013749999459832907 0.026100000366568565 0.042499999050050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; visual mesh filename=meshes/kistar/finger_link_1.STL
- link index_link_2: geometry collision box size=0.013750000391155481 0.02599999960511923 0.0356988441199064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; visual mesh filename=meshes/kistar/finger_link_2.STL
- link index_tip: geometry collision mesh filename=meshes/kistar/finger_tip.STL; visual mesh filename=meshes/kistar/finger_tip.STL
- link middle_basemotor: geometry visual mesh filename=meshes/kistar/finger_basemotor.STL
- link middle_link_0: geometry collision box size=0.026000000536441803 0.026000000536441803 0.028453040402382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; visual mesh filename=meshes/kistar/finger_link_0.STL
- link middle_link_1: geometry collision box size=0.013749999459832907 0.026100000366568565 0.042499999050050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; visual mesh filename=meshes/kistar/finger_link_1.STL
- link middle_link_2: geometry collision box size=0.013750000391155481 0.02599999960511923 0.0356988441199064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; visual mesh filename=meshes/kistar/finger_link_2.STL
- link middle_tip: geometry collision mesh filename=meshes/kistar/finger_tip.STL; visual mesh filename=meshes/kistar/finger_tip.STL
- link mount: geometry collision cylinder length=0.00999999955296517 radius=0.019931690767407417; visual mesh filename=meshes/kistar/mount.STL
- link palm: geometry collision box size=0.04700000025331974 0.0895427018404007 0.08685353584587574; visual mesh filename=meshes/kistar/palm02.STL
- link ring_basemotor: geometry visual mesh filename=meshes/kistar/finger_basemotor.STL
- link ring_link_0: geometry collision box size=0.026000000536441803 0.026000000536441803 0.028453040402382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; visual mesh filename=meshes/kistar/finger_link_0.STL
- link ring_link_1: geometry collision box size=0.013749999459832907 0.026100000366568565 0.042499999050050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; visual mesh filename=meshes/kistar/finger_link_1.STL
- link ring_link_2: geometry collision box size=0.013750000391155481 0.02599999960511923 0.0356988441199064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; visual mesh filename=meshes/kistar/finger_link_2.STL
- link ring_tip: geometry collision mesh filename=meshes/kistar/finger_tip.STL; visual mesh filename=meshes/kistar/finger_tip.STL
- link thumb_basemotor: geometry visual mesh filename=meshes/kistar/thumb_basemotor.STL
- link thumb_link_0: geometry collision box size=0.026284214574843645 0.026000000536441803 0.040484629105776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; visual mesh filename=meshes/kistar/thumb_link_0.STL
- link thumb_link_1: geometry collision box size=0.013000000268220901 0.026000000536441803 0.014479377320036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; visual mesh filename=meshes/kistar/thumb_link_1.STL
- link thumb_link_2: geometry collision box size=0.013749999459832907 0.026100000366568565 0.042499997187405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; visual mesh filename=meshes/kistar/thumb_link_2.STL
- link thumb_tip: geometry collision mesh filename=meshes/kistar/thumb_tip.STL; visual mesh filename=meshes/kistar/thumb_tip.STL
Joints:
- removed joint index_sensor_0
- removed joint index_sensor_1
- removed joint index_sensor_2
- removed joint middle_sensor_0
- removed joint middle_sensor_1
- removed joint middle_sensor_2
- removed joint ring_sensor_0
- removed joint ring_sensor_1
- removed joint ring_sensor_2
- removed joint thumb_sensor_0
- removed joint thumb_sensor_1
