Commit message: Add: Kistar urdf and configuration

File: grasp_generation/kistar/kistar.urdf (robot description, URDF)
Before this commit: robot kistar_hand, 22 links, 21 joints
Links:
- link index_basemotor: geometry collision box size=0.028149999655596912 0.01919999998062849 0.0240000002086162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; visual mesh filename=meshes/kistar/finger_basemotor.STL
- link middle_basemotor: geometry collision box size=0.028149999655596912 0.01919999998062849 0.0240000002086162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; visual mesh filename=meshes/kistar/finger_basemotor.STL
- link mount: geometry collision mesh filename=meshes/kistar/mount.STL; visual mesh filename=meshes/kistar/mount.STL
- link ring_basemotor: geometry collision box size=0.028149999655596912 0.01919999998062849 0.0240000002086162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; visual mesh filename=meshes/kistar/finger_basemotor.STL
- link thumb_basemotor: geometry collision box size=0.02400000027120114 0.01919999998062849 0.024000000208616257; visual mesh filename=meshes/kistar/thumb_basemotor.STL
